File: redox-f14/pcb/wingxx_receiver_kicad_files_v3/wing-receiver-lite-case.kicad_pcb (KiCad board)
At the start: 2 copper layers, 74.9 x 47.5 mm, 29 parts, among them U1 ATmega32U4-AU, X1 Crystal_GND24

Commit message: update to new style
Other:
- board size 74.9 x 47.5 mm -> 80.5 x 50.5 mm
Changed lines of the file:
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@@
   (general
     (thickness 1.6)
-    (drawings 46)
+    (drawings 57)
     (tracks 325)
     (zones 0)
@@
     (0 F.Cu signal hide)
     (31 B.Cu signal hide)
-    (32 B.Adhes user hide)
-    (33 F.Adhes user hide)
-    (34 B.Paste user hide)
-    (35 F.Paste user hide)
+    (32 B.Adhes user)
+    (33 F.Adhes user)
+    (34 B.Paste user)
+    (35 F.Paste user)
     (36 B.SilkS user)
-    (37 F.SilkS user hide)
-    (38 B.Mask user hide)
-    (39 F.Mask user hide)
+    (37 F.SilkS user)
+    (38 B.Mask user)
+    (39 F.Mask user)
     (40 Dwgs.User user)
-    (41 Cmts.User user hide)
-    (42 Eco1.User user hide)
-    (43 Eco2.User user hide)
+    (41 Cmts.User user)
+    (42 Eco1.User user)
+    (43 Eco2.User user)
     (44 Edge.Cuts user)
-    (45 Margin user hide)
-    (46 B.CrtYd user hide)
-    (47 F.CrtYd user hide)
-    (48 B.Fab user hide)
-    (49 F.Fab user hide)
+    (45 Margin user)
+    (46 B.CrtYd user)
+    (47 F.CrtYd user)
+    (48 B.Fab user)
+    (49 F.Fab user)
   )
   (setup
@@
     )
   )
+  (gr_arc (start 91.44 133.35) (end 91.44 132.334) (angle -180) (layer Edge.Cuts) (width 0.1))
+  (gr_arc (start 68.326 133.35) (end 68.326 134.366) (angle -180) (layer Edge.Cuts) (width 0.1))
+  (gr_arc (start 91.186 96.52) (end 91.186 95.504) (angle -180) (layer Edge.Cuts) (width 0.1))
+  (gr_arc (start 68.326 96.52) (end 68.326 97.536) (angle -180) (layer Edge.Cuts) (width 0.1))
+  (gr_line (start 85.598 91.948) (end 96.774 91.948) (layer Edge.Cuts) (width 0.1))
+  (gr_line (start 84.582 92.71) (end 85.598 91.948) (layer Edge.Cuts) (width 0.1))
+  (gr_line (start 71.12 142.494) (end 88.9 142.494) (layer Edge.Cuts) (width 0.1))
+  (gr_line (start 96.774 91.948) (end 96.774 136.652) (layer Edge.Cuts) (width 0.1))
+  (gr_line (start 73.914 91.948) (end 74.93 92.71) (layer Edge.Cuts) (width 0.1))
+  (gr_line (start 73.914 91.948) (end 62.738 91.948) (layer Edge.Cuts) (width 0.1))
+  (gr_line (start 62.738 91.948) (end 62.738 136.652) (layer Edge.Cuts) (width 0.1))
   (dimension 47.244 (width 0.15) (layer Dwgs.User)
     (gr_text "47.244 mm" (at 113.254 116.078 90) (layer Dwgs.User)

Commit message: new receiver
Parts:
- added RESET1: SW_SPST, Button_Switch_SMD:SW_SPST_CK_RS282G05A3, B.Cu at (79.8, 105.9)
Other:
- board size 80.5 x 50.5 mm -> 248.7 x 121.2 mm
