File: redox-f14/pcb/wingxx_receiver_kicad_files_v2/wingxx-receiver-case-v4.kicad_pcb (KiCad board)
At the start: 2 copper layers, 198.1 x 335.3 mm, 16 parts, among them K1 KEYSW-redox_rev1-rescue, K11 KEYSW-redox_rev1-rescue, K12 KEYSW-redox_rev1-rescue, K13 KEYSW-redox_rev1-rescue, K14 KEYSW-redox_rev1-rescue, K2 KEYSW-redox_rev1-rescue, K21 KEYSW-redox_rev1-rescue, K22 KEYSW-redox_rev1-rescue, K23 KEYSW-redox_rev1-rescue, K24 KEYSW-redox_rev1-rescue, K3 KEYSW-redox_rev1-rescue, K31 KEYSW-redox_rev1-rescue, K32 KEYSW-redox_rev1-rescue, K33 KEYSW-redox_rev1-rescue, K34 KEYSW-redox_rev1-rescue, K4 KEYSW-redox_rev1-rescue

Commit message: add receiver v2.5
Parts:
- added SW1: SW_Left, v60_kicad_files:SW_SPDT_MSS22D18G2, B.Cu at (55.3, 126.0)
Other:
- outline, holes or cut-outs redrawn
Changed lines of the file:
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@@
   (general
     (thickness 1.6)
-    (drawings 116)
+    (drawings 120)
     (tracks 0)
     (zones 0)
-    (modules 16)
+    (modules 17)
     (nets 1)
   )
@@
     (uvia_drill 0.1)
   )
+  (module v60_kicad_files:SW_SPDT_MSS22D18G2 (layer B.Cu)
+    (at 55.3085 126.0475 270)
+    (descr http://www.ckswitches.com/media/1422/js.pdf)
+    (tags "switch spdt")
+    (attr smd)
+    (fp_text reference SW1 (at 0 4.8 270) (layer B.SilkS)
+      (effects (font (size 1 1) (thickness 0.15)) (justify mirror))
+    )
+    (fp_text value SW_Left (at 0 2.9 270) (layer B.Fab)
+      (effects (font (size 1 1) (thickness 0.15)) (justify mirror))
+    )
+    (fp_line (start -5 2.25) (end -5 2.25) (layer B.CrtYd) (width 0.05))
+    (fp_line (start -3.5 2.25) (end -5 2.25) (layer B.CrtYd) (width 0.05))
+    (fp_line (start -3.5 4.5) (end -3.5 2.25) (layer B.CrtYd) (width 0.05))
+    (fp_line (start 3.5 4.5) (end -3.5 4.5) (layer B.CrtYd) (width 0.05))
+    (fp_line (start 3.5 2.25) (end 3.5 4.5) (layer B.CrtYd) (width 0.05))
+    (fp_line (start 5 2.25) (end 3.5 2.25) (layer B.CrtYd) (width 0.05))
+    (fp_line (start 5 -2.25) (end 5 2.25) (layer B.CrtYd) (width 0.05))
+    (fp_line (start 3.25 -2.25) (end 5 -2.25) (layer B.CrtYd) (width 0.05))
+    (fp_line (start 3.25 -2.5) (end 3.25 -2.25) (layer B.CrtYd) (width 0.05))
+    (fp_line (start 2.5 -2.5) (end 3.25 -2.5) (layer B.CrtYd) (width 0.05))
+    (fp_line (start 2.5 -4.25) (end 2.5 -2.5) (layer B.CrtYd) (width 0.05))
+    (fp_line (start -2.5 -4.25) (end 2.5 -4.25) (layer B.CrtYd) (width 0.05))
+    (fp_line (start -2.5 -2.75) (end -2.5 -4.25) (layer B.CrtYd) (width 0.05))
+    (fp_line (start -3.25 -2.75) (end -2.5 -2.75) (layer B.CrtYd) (width 0.05))
+    (fp_line (start -3.25 -2.25) (end -3.25 -2.75) (layer B.CrtYd) (width 0.05))
+    (fp_line (start -5 -2.25) (end -3.25 -2.25) (layer B.CrtYd) (width 0.05))
+    (fp_line (start -5 2.25) (end -5 -2.25) (layer B.CrtYd) (width 0.05))
+    (fp_line (start -2 -1.8) (end -2 -1.8) (layer B.Fab) (width 0.1))
+    (fp_line (start -0.5 -1.8) (end -0.5 -3.8) (layer B.Fab) (width 0.1))
+    (fp_line (start -4.6 -1.9) (end -4.6 -1.9) (layer B.SilkS) (width 0.12))
+    (fp_line (start -3.2 -1.9) (end -4.6 -1.9) (layer B.SilkS) (width 0.12))
+    (fp_line (start -0.7 -1.9) (end -1.8 -1.9) (layer B.SilkS) (width 0.12))
+    (fp_line (start 1.8 -1.9) (end 0.7 -1.9) (layer B.SilkS) (width 0.12))
+    (fp_line (start 4.6 -1.9) (end 3.2 -1.9) (layer B.SilkS) (width 0.12))
+    (fp_line (start 2.8 -1.8) (end 2.8 -1.8) (layer B.Fab) (width 0.1))
+    (fp_line (start 2.8 -2.1) (end 2.8 -1.8) (layer B.Fab) (width 0.1))
+    (fp_line (start 2.2 -2.1) (end 2.8 -2.1) (layer B.Fab) (width 0.1))
+    (fp_line (start 2.2 -1.8) (end 2.2 -2.1) (layer B.Fab) (width 0.1))
+    (fp_line (start -2.8 -1.8) (end -2.8 -1.8) (layer B.Fab) (width 0.1))
+    (fp_line (start -2.8 -2.1) (end -2.8 -1.8) (layer B.Fab) (width 0.1))
+    (fp_line (start -2.2 -2.1) (end -2.8 -2.1) (layer B.Fab) (width 0.1))
+    (fp_line (start -2.2 -1.8) (end -2.2 -2.1) (layer B.Fab) (width 0.1))
+    (fp_line (start -0.3 -1.8) (end -0.3 -1.8) (layer B.Fab) (width 0.1))
+    (fp_line (start -0.3 -2.1) (end -0.3 -1.8) (layer B.Fab) (width 0.1))
+    (fp_line (start 0.3 -1.8) (end 0.3 -2.1) (layer B.Fab) (width 0.1))
+    (fp_line (start -1.8 1.9) (end -1.8 1.9) (layer B.SilkS) (width 0.12))
+    (fp_line (start -0.7 1.9) (end -1.8 1.9) (layer B.SilkS) (width 0.12))
+    (fp_line (start 0.7 1.9) (end 0.7 1.9) (layer B.SilkS) (width 0.12))
+    (fp_line (start 1.8 1.9) (end 0.7 1.9) (layer B.SilkS) (width 0.12))
+    (fp_line (start -4.6 1.9) (end -3.2 1.9) (layer B.SilkS) (width 0.12))
+    (fp_line (start -4.6 -1.9) (end -4.6 1.9) (layer B.SilkS) (width 0.12))
+    (fp_line (start 4.6 1.9) (end 4.6 -1.9) (layer B.SilkS) (width 0.12))
+    (fp_line (start 3.2 1.9) (end 4.6 1.9) (layer B.SilkS) (width 0.12))
+    (fp_line (start -1.5 -1.8) (end -1.5 -1.8) (layer B.Fab) (width 0.1))
+    (fp_text user %R (at 0 0 270) (layer B.Fab)
+      (effects (font (size 1 1) (thickness 0.15)) (justify mirror))
+    )
+    (fp_line (start -4.5 -1.8) (end -4.5 -1.8) (layer B.Fab) (width 0.1))
+    (fp_line (start -4.5 1.8) (end -4.5 -1.8) (layer B.Fab) (width 0.1))
+    (fp_line (start -4.5 -1.8) (end -4.5 -1.8) (layer B.Fab) (width 0.1))
+    (fp_line (start -4.4 -1.8) (end -4.5 -1.8) (layer B.Fab) (width 0.1))
+    (fp_line (start 4.5 -1.8) (end -4.4 -1.8) (layer B.Fab) (width 0.1))
+    (fp_line (start 4.5 1.8) (end 4.5 -1.8) (layer B.Fab) (width 0.1))
+    (fp_line (start -4.5 1.8) (end 4.5 1.8) (layer B.Fab) (width 0.1))
+    (pad 6 smd rect (at 2.5 -2.75 90) (size 1.25 2.5) (layers B.Cu B.Paste B.Mask))
+    (pad 5 smd rect (at 0 -2.75 90) (size 1.25 2.5) (layers B.Cu B.Paste B.Mask))
+    (pad 4 smd rect (at -2.5 -2.75 90) (size 1.25 2.5) (layers B.Cu B.Paste B.Mask))
+    (pad 3 smd rect (at 2.5 2.75 270) (size 1.25 2.5) (layers B.Cu B.Paste B.Mask))
+    (pad 2 smd rect (at 0 2.75 270) (size 1.25 2.5) (layers B.Cu B.Paste B.Mask))
+    (pad 1 smd rect (at -2.5 2.75 270) (size 1.25 2.5) (layers B.Cu B.Paste B.Mask))
+    (model ${KISYS3DMOD}/Button_Switch_SMD.3dshapes/SW_SPDT_CK-JS102011SAQN.wrl
+      (at (xyz 0 0 0))
+      (scale (xyz 1 1 1))
+      (rotate (xyz 0 0 0))
+    )
+  )
   (module pcb:SW_Cherry_MX_1.00u_PCB (layer F.Cu)
     (at 55.245 2.3812)
@@
     )
   )
+  (gr_line (start 56.642 122.428) (end 56.642 129.54) (layer Edge.Cuts) (width 0.1))
+  (gr_line (start 53.721 129.54) (end 53.721 122.428) (layer Edge.Cuts) (width 0.1))
+  (gr_line (start 53.721 122.428) (end 56.642 122.428) (layer Edge.Cuts) (width 0.1))
+  (gr_line (start 56.642 129.54) (end 53.721 129.54) (layer Edge.Cuts) (width 0.1))
   (gr_line (start 148.59 50.165) (end 224.79 50.165) (layer Edge.Cuts) (width 0.1))
   (gr_line (start 224.79 -26.67) (end 148.59 -26.67) (layer Edge.Cuts) (width 0.1))
