File: redox-f14/pcb/wingxx_receiver_kicad_files_v2/wingxx-receiver-v4.kicad_pcb (KiCad board)
At the start: 2 copper layers, 78.7 x 90.2 mm, 61 parts, among them K1 KEYSW-redox_rev1-rescue, K11 KEYSW-redox_rev1-rescue, K12 KEYSW-redox_rev1-rescue, K13 KEYSW-redox_rev1-rescue, K14 KEYSW-redox_rev1-rescue, K2 KEYSW-redox_rev1-rescue, K21 KEYSW-redox_rev1-rescue, K22 KEYSW-redox_rev1-rescue, K23 KEYSW-redox_rev1-rescue, K24 KEYSW-redox_rev1-rescue, K3 KEYSW-redox_rev1-rescue, K31 KEYSW-redox_rev1-rescue, K32 KEYSW-redox_rev1-rescue, K33 KEYSW-redox_rev1-rescue, K34 KEYSW-redox_rev1-rescue, K4 KEYSW-redox_rev1-rescue, U1 ATmega32U4-AU, X1 Crystal_GND24

Commit message: new receiver
Parts:
- D1, D11, D12, D13, D14, D2, D21, D22, D23, D24, D3, D31, D32, D33, D34, D4: footprint pcb:D3_SMD_Back -> pcb:D3_SMD_Front; moved to B.Cu
Routing:
- net col2: track 96.0 -> 132.9 mm
- net GND: track 375.6 -> 402.5 mm, vias 3 -> 0
- net VCC: track 78.3 -> 104.0 mm
- net +5V: track 156.7 -> 175.2 mm, vias 1 -> 2
- net row3: track 118.6 -> 130.3 mm
- net +3.3V: track 141.8 -> 148.8 mm
- net Net-(D6-Pad3): track 37.4 -> 31.1 mm
- net col1: track 82.6 -> 87.2 mm, vias 4 -> 3
- net RGB_DATA: track 69.3 -> 66.7 mm
- net row1: track 95.3 -> 96.6 mm
- net POF5: track 41.3 -> 42.6 mm
- net Net-(R5-Pad2): track 36.4 -> 37.5 mm, vias 2 -> 0
- net Net-(C3-Pad1): track 19.3 -> 18.4 mm
- net POF4: track 41.4 -> 42.2 mm
- net row0: track 98.7 -> 99.4 mm
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
Commit message: add receiver v2.5
Parts:
- removed V_REG1: LD1117S33CTR, redox_w_receiver_footprints:SOT-223
- added IC2: XC6206P332MR, XC6206P332MR:SOT95P280X130-3N, B.Cu at (127.1, 62.3)
- C11, C12: value 10uF -> 1uF
- moved ConnFemale_Underglow1 101.4 mm to (81.3, 145.4)
- moved PROGR_HEADER2 43.7 mm to (76.8, 94.0), turned to 0 degrees
- moved C11 39.9 mm to (134.3, 61.1), turned to 0 degrees
- moved C3 37.2 mm to (118.1, 94.6)
- moved R5 36.7 mm to (118.1, 97.8)
- moved R6 36.7 mm to (118.1, 101.0)
- moved C12 32.1 mm to (134.3, 64.0), turned to 0 degrees
- moved PROGR_HEADER1 20.9 mm to (101.0, 145.4), turned to 270 degrees
- moved R11 8.51 mm to (98.7, 141.0), turned to 180 degrees
- moved R13 7.92 mm to (98.7, 133.3), turned to 180 degrees
- moved R12 6.21 mm to (98.7, 137.2), turned to 180 degrees
Connections:
- C11 pad 1: VCC -> GND
- C11 pad 2: GND -> VCC
- C12 pad 1: +3.3V -> GND
- C12 pad 2: GND -> +3.3V
Routing:
- net GND: track 402.5 -> 318.2 mm, vias 0 -> 6
- net VCC: track 104.0 -> 55.4 mm, vias 4 -> 2
- net +3.3V: track 148.8 -> 110.1 mm, vias 0 -> 1
- net col2: track 132.9 -> 95.3 mm
- net row3: track 130.3 -> 99.8 mm, vias 2 -> 3
- net POF4: track 42.2 -> 13.2 mm, vias 1 -> 0
- net POF0: track 42.2 -> 13.6 mm, vias 1 -> 0
- net POF5: track 42.6 -> 14.1 mm, vias 1 -> 0
- net POF1: track 41.0 -> 13.1 mm, vias 1 -> 0
- net RGB_DATA: track 66.7 -> 46.4 mm
- net Net-(D33-Pad2): track 28.0 -> 13.0 mm
- net Net-(D31-Pad2): track 13.0 -> 27.6 mm
- net Net-(R2-Pad2): track 36.4 -> 49.5 mm
- net SWCLK: track 42.3 -> 30.2 mm, vias 0 -> 1
- net +5V: track 175.2 -> 164.9 mm, vias 2 -> 4
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- added copper zone on B.Cu, net (none)
- added copper zone on F.Cu, net (none)
Other:
- outline, holes or cut-outs redrawn
