File: redox-f14/pcb/wingxx_receiver_kicad_files_v2/wingxx-receiver-v4.sch (KiCad schematic (older format))
At the start: 79 parts, among them K1 KEYSW-redox_rev1-rescue, K11 KEYSW-redox_rev1-rescue, K12 KEYSW-redox_rev1-rescue, K13 KEYSW-redox_rev1-rescue, K14 KEYSW-redox_rev1-rescue, K15 KEYSW-redox_rev1-rescue, K2 KEYSW-redox_rev1-rescue, K21 KEYSW-redox_rev1-rescue, K22 KEYSW-redox_rev1-rescue, K23 KEYSW-redox_rev1-rescue, K24 KEYSW-redox_rev1-rescue, K25 KEYSW-redox_rev1-rescue, K3 KEYSW-redox_rev1-rescue, K31 KEYSW-redox_rev1-rescue, K32 KEYSW-redox_rev1-rescue, K33 KEYSW-redox_rev1-rescue, K34 KEYSW-redox_rev1-rescue, K35 KEYSW-redox_rev1-rescue, K4 KEYSW-redox_rev1-rescue, K41 KEYSW-redox_rev1-rescue, K42 KEYSW-redox_rev1-rescue, K43 KEYSW-redox_rev1-rescue, K44 KEYSW-redox_rev1-rescue, K45 KEYSW-redox_rev1-rescue, K5 KEYSW-redox_rev1-rescue, U1 ATmega32U4-AU, X1 Crystal_GND24

Commit message: add receiver v2.5
Parts:
- removed V_REG1: LD1117S33CTR, redox_w_receiver_footprints:SOT-223, symbol redox-receiver-rescue:LD1117S33CTR-dk_PMIC-Voltage-Regulators-Linear
- added IC2: XC6206P332MR, XC6206P332MR:SOT95P280X130-3N, symbol f14_v60_v2-cache:f14_v60-rescue_XC6206P332MR-XC6206P332MR
- C11, C12: value 10uF -> 1uF
- D1, D11, D12, D13, D14, D15, D2, D21, D22, D23, D24, D25, D3, D31, D32, D33, D34, D35, D4, D41, D42, D43, D44, D45, D5: footprint pcb:D3_SMD_Back -> pcb:D3_SMD_Front
Connections:
- net +3.3V: now also C12.2, IC2.2 (VOUT); no longer C12.1
- net GND: now also C11.1, C12.1, IC2.1 (VSS); no longer C11.2, C12.2
- net VCC: now also C11.2, IC2.3 (VIN); no longer C11.1
