File: redox-f14/pcb/wingxx_receiver_kicad_files_v2/wingxx-receiver-v4-wiredcut.sch (KiCad schematic (older format))
At the start: 27 parts, among them IC2 XC6206P332MR, U1 ATmega32U4-AU, X1 Crystal_GND24

Commit message: new receiver
Parts:
- removed C11, C12: 1uF, Capacitor_SMD:C_0805_2012Metric_Pad1.15x1.40mm_HandSolder, symbol Device:C
- removed IC2: XC6206P332MR, SOT95P280X130-3N, symbol XC6206P332MR:XC6206P332MR
- removed PROGR_HEADER1: Conn_01x04_Female, Connector_PinHeader_2.54mm:PinHeader_1x04_P2.54mm_Vertical, symbol wingxx-receiver-v4-rescue:Conn_01x04-Connector_Generic-redox-receiver-rescue
- removed R11, R12, R13: 1.5K, Resistor_SMD:R_0805_2012Metric_Pad1.15x1.40mm_HandSolder, symbol wingxx-receiver-v4-rescue:R-Device-redox-receiver-rescue
- removed nrf1: E73-nrf51822, wingxx-receiver:E73-nrf51822-Module, symbol wingxx-receiver-v4-rescue:E73-nrf51822-redox-receiver-rescue
- RESET1: symbol wingxx-receiver-v4-rescue:SW_SPST-Switch-redox-receiver-rescue -> redox-receiver-rescue:SW_SPST-Switch
- USB1: symbol wingxx-receiver-v4-rescue:HRO-TYPE-C-31-M-12-Type-C -> Type-C:HRO-TYPE-C-31-M-12
Connections:
- net labels added: POF0, POF1, POF4, POF5, RGB_DATA, col0, col1, col2, col3, col4, row0, row1, row2, row3, row4
- net labels removed: +3.3V, SWCLK, SWDIO, TXODIV
- wire segments 123 -> 98
- no-connect marks 53 -> 3
